File: Eagle/Bachelor/main_schematic.sch (EAGLE design)
At the start: 113 parts, among them Q2 16MHz, SW7 SPST_TACT-EVQQ2, SW8 SPST_TACT-EVQQ2, SW9 SPST_TACT-EVQQ2, U1 ATMEGA32U4-AU, U2 ADP2302ARDZ-5.0-R7, X1 MICROMATCH-4, X2 MICROMATCH-4, X3 MICROMATCH-4

Commit message: Done
Connections:
- net ANALOG renamed VREF
- net HIGH_VOLTAGE renamed 12VINPUT
- net KILL1 renamed STOP1
- net KILL2 renamed STOP2
- net KILL3 renamed STOP3
- net KILL4 renamed STOP4
- net KILL5 renamed STOP5
- net KILL6 renamed STOP6
