File: Eagle/Bachelor/main_schematic_correction.sch (EAGLE design)
At the start: 112 parts, among them Q2 16MHz, SW7 SPST_TACT-EVQQ2, SW8 SPST_TACT-EVQQ2, SW9 SPST_TACT-EVQQ2, U1 ATMEGA32U4-AU, U2 ADP2302ARDZ-5.0-R7, X1 MICROMATCH-4, X2 MICROMATCH-4, X3 MICROMATCH-4

Commit message: Done
Connections:
- new net N$134: C52.2
- new net N$135: C53.2
- new net N$136: C54.2
- net VCC: no longer C52.2, C53.2, C54.2
Changed lines of the file:
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@@
 <part name="GND59" library="supply1" deviceset="GND" device=""/>
 <part name="C52" library="rcl" deviceset="C-EU" device="C0603K" value="100nF"/>
-<part name="P+20" library="supply1" deviceset="VCC" device=""/>
 <part name="C53" library="rcl" deviceset="C-EU" device="C0603K" value="100nF"/>
-<part name="P+21" library="supply1" deviceset="VCC" device=""/>
 <part name="C54" library="rcl" deviceset="C-EU" device="C0603K" value="100nF"/>
-<part name="P+22" library="supply1" deviceset="VCC" device=""/>
 <part name="P+23" library="supply1" deviceset="VCC" device=""/>
 <part name="X5" library="con-wago-508" deviceset="W237-04P" device=""/>
@@
 <attribute name="VALUE" x="117.348" y="30.353" size="1.778" layer="96"/>
 </instance>
-<instance part="P+20" gate="VCC" x="111.76" y="30.48" smashed="yes">
-<attribute name="VALUE" x="114.3" y="32.512" size="1.778" layer="96" rot="R180"/>
-</instance>
 <instance part="C53" gate="G$1" x="119.38" y="-30.48" smashed="yes" rot="R270">
 <attribute name="NAME" x="119.38" y="-30.353" size="1.778" layer="95"/>
 <attribute name="VALUE" x="117.348" y="-28.067" size="1.778" layer="96"/>
 </instance>
-<instance part="P+21" gate="VCC" x="111.76" y="-27.94" smashed="yes">
-<attribute name="VALUE" x="114.3" y="-25.908" size="1.778" layer="96" rot="R180"/>
-</instance>
 <instance part="C54" gate="G$1" x="119.38" y="-83.82" smashed="yes" rot="R270">
 <attribute name="NAME" x="119.38" y="-83.693" size="1.778" layer="95"/>
 <attribute name="VALUE" x="117.348" y="-81.407" size="1.778" layer="96"/>
-</instance>
-<instance part="P+22" gate="VCC" x="111.76" y="-81.28" smashed="yes">
-<attribute name="VALUE" x="114.3" y="-79.248" size="1.778" layer="96" rot="R180"/>
 </instance>
 <instance part="P+23" gate="VCC" x="-45.72" y="22.86"/>
@@
 </segment>
 <segment>
-<pinref part="C52" gate="G$1" pin="2"/>
-<wire x1="114.3" y1="27.94" x2="111.76" y2="27.94" width="0.1524" layer="91"/>
-<pinref part="P+20" gate="VCC" pin="VCC"/>
-</segment>
-<segment>
-<pinref part="C53" gate="G$1" pin="2"/>
-<wire x1="114.3" y1="-30.48" x2="111.76" y2="-30.48" width="0.1524" layer="91"/>
-<pinref part="P+21" gate="VCC" pin="VCC"/>
-</segment>
-<segment>
-<pinref part="C54" gate="G$1" pin="2"/>
-<wire x1="114.3" y1="-83.82" x2="111.76" y2="-83.82" width="0.1524" layer="91"/>
-<pinref part="P+22" gate="VCC" pin="VCC"/>
-</segment>
-<segment>
 <pinref part="F1" gate="G$1" pin="P$2"/>
 <wire x1="-66.04" y1="-45.72" x2="-55.88" y2="-45.72" width="0.1524" layer="91"/>
@@
 <wire x1="251.46" y1="-73.66" x2="251.46" y2="-71.12" width="0.1524" layer="91"/>
 <junction x="251.46" y="-71.12"/>
+<label x="106.68" y="-83.82" size="1.27" layer="95" rot="R180" xref="yes"/>
 </segment>
 <segment>
@@
 <wire x1="251.46" y1="38.1" x2="251.46" y2="40.64" width="0.1524" layer="91"/>
 <junction x="251.46" y="40.64"/>
-</segment>
-</net>
+<label x="109.22" y="27.94" size="1.27" layer="95" rot="R180" xref="yes"/>
+<label x="106.68" y="-30.48" size="1.27" layer="95" rot="R180" xref="yes"/>
+</segment>
+</net>
+<net name="N$134" class="0">
+<segment>
+<pinref part="C52" gate="G$1" pin="2"/>
+<wire x1="109.22" y1="27.94" x2="114.3" y2="27.94" width="0.1524" layer="91"/>
+</segment>
+</net>
+<net name="N$135" class="0">
+<segment>
+<pinref part="C53" gate="G$1" pin="2"/>
+<wire x1="106.68" y1="-30.48" x2="114.3" y2="-30.48" width="0.1524" layer="91"/>
+</segment>
+</net>
+<net name="N$136" class="0">
+<segment>
+<pinref part="C54" gate="G$1" pin="2"/>
+<wire x1="106.68" y1="-83.82" x2="114.3" y2="-83.82" width="0.1524" layer="91"/>
+</segment>
+</net>
